File: board/DO6TS1A.kicad_pcb (KiCad board)
At the start: 2 copper layers, 60 x 55 mm, 29 parts, among them U1 RT9193, U2 HLK-PM01, U3 PCF8574, U4 ESP-12, X1 ESP-PROG

Commit message: WIP
Parts:
- C3: value 47u -> 1u
- moved D1 66.6 mm to (73.0, 93.1), turned to 90 degrees
- moved R3 59.9 mm to (73.0, 100.0), turned to 90 degrees
- moved D2 46.2 mm to (77.0, 96.9), turned to 90 degrees
- moved R4 37.7 mm to (76.0, 103.0), turned to 90 degrees
- moved C6 26.6 mm to (107.0, 110.0), turned to 90 degrees
- moved R7 25.7 mm to (95.0, 128.1), turned to 270 degrees
- moved R8 25.3 mm to (89.0, 128.1), turned to 270 degrees
- moved C7 22.2 mm to (92.0, 128.0), turned to 90 degrees
- moved C5 16.6 mm to (111.0, 110.0), turned to 90 degrees
- moved C4 11.4 mm to (109.0, 110.0), turned to 90 degrees
- moved L1 8.15 mm to (101.0, 95.0)
- moved R1 6.05 mm to (114.0, 110.0), turned to 270 degrees
- moved R9 5.36 mm to (105.0, 103.0), turned to 90 degrees
- moved C3 5.00 mm to (101.0, 92.0), turned to 180 degrees
- moved R6 2.76 mm to (102.0, 103.0), turned to 90 degrees
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- renumbered C8 to C4, C9 to C5, C4 to C6, D2 to D1, D3 to D2, D1 to D3, R3 to R2, R2 to R3, U3 to U1, U1 to U2, U2 to U3
Routing:
- net Net-(D2-Pad1): track 0.00 -> 0.71 mm

Commit message: WIP
Parts:
- moved R4 12.1 mm to (85.0, 95.0)
- moved R3 12.0 mm to (85.0, 101.0), turned to 270 degrees
- moved D1 12.0 mm to (82.0, 101.0)
- moved D2 5.39 mm to (82.0, 94.9), turned to 270 degrees
- moved MAINS1 5.00 mm to (127.0, 136.0)
Connections:
- D1 pad 2: Net-(D1-Pad2) -> VCC
- D2 pad 2: Net-(D2-Pad2) -> VCC
- R3 pad 1: Net-(D1-Pad2) -> Net-(R3-Pad1)
- R3 pad 2: VCC -> Net-(D1-Pad1)
- R4 pad 1: Net-(D2-Pad2) -> Net-(R4-Pad1)
- R4 pad 2: VCC -> Net-(D2-Pad1)
- U1 pad 11: Net-(D1-Pad1) -> Net-(R3-Pad1)
- U1 pad 12: Net-(D2-Pad1) -> Net-(R4-Pad1)
Routing:
- net VCC: track 0.00 -> 112.3 mm
- net /5V: track 0.00 -> 78.4 mm
- net /SDA: track 0.00 -> 46.8 mm, vias 0 -> 2
- net /SCL: track 0.00 -> 45.5 mm, vias 0 -> 4
- net Net-(R3-Pad1): track 0.00 -> 44.0 mm, vias 0 -> 2
- net Net-(R4-Pad1): track 0.00 -> 38.8 mm, vias 0 -> 2
- net /ESP/RESET: track 0.00 -> 36.8 mm
- net /ESP/5V-PROG: track 0.00 -> 33.4 mm, vias 0 -> 2
- net GND: track 0.00 -> 31.7 mm, vias 0 -> 9
- net /ESP/GPIO4: track 0.00 -> 31.4 mm, vias 0 -> 1
- net /ESP/5V-MAINS: track 0.00 -> 24.1 mm
- net Net-(DO1-Pad9): track 0.00 -> 21.5 mm
- net Net-(DO1-Pad11): track 0.00 -> 21.0 mm, vias 0 -> 2
- net /ESP/GPIO0: track 0.00 -> 13.2 mm, vias 0 -> 2
- net /ESP/MAINS-2: track 0.00 -> 13.0 mm
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- added copper zone on B.Cu, net GND

Commit message: WIP
Other:
- board text added: "230VAC"
- board text added: "Address:"
- board text added: "CC-BY-SA"
- board text added: "DEVICE.FARM"
- board text added: "DO6TS1A 1.0"
- board text added: "ESPP"
- board text added: "I2C"
- board text added: "TS:GND/DATA/3V3"
- board text added: "TTL OUT"
Changed lines of the file:
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@@
     (area 79.949999 84.949999 140.050001 140.050001)
     (thickness 1.6)
-    (drawings 7)
-    (tracks 260)
+    (drawings 17)
+    (tracks 258)
     (zones 0)
     (modules 29)
@@
     (tags "capacitor 0805")
     (attr smd)
-    (fp_text reference C1 (at 0 -1.5 270) (layer F.SilkS)
+    (fp_text reference C1 (at 2.5 -0.5 360) (layer F.SilkS)
       (effects (font (size 1 1) (thickness 0.15)))
     )
@@
     (tags "capacitor 0805")
     (attr smd)
-    (fp_text reference C2 (at 0 -1.5 180) (layer F.SilkS)
+    (fp_text reference C2 (at 3 0 180) (layer F.SilkS)
       (effects (font (size 1 1) (thickness 0.15)))
     )
@@
     (tags "capacitor 0805")
     (attr smd)
-    (fp_text reference C3 (at 0 -1.5 180) (layer F.SilkS)
+    (fp_text reference C3 (at 3 0 180) (layer F.SilkS)
       (effects (font (size 1 1) (thickness 0.15)))
     )
@@
     (tags "capacitor 0805")
     (attr smd)
-    (fp_text reference C6 (at 0 -1.5 90) (layer F.SilkS)
+    (fp_text reference C6 (at 3.5 0 180) (layer F.SilkS)
       (effects (font (size 1 1) (thickness 0.15)))
     )
@@
     (tags "capacitor 0805")
     (attr smd)
-    (fp_text reference C7 (at 0 -1.5 90) (layer F.SilkS)
+    (fp_text reference C7 (at 2.5 0 180) (layer F.SilkS)
       (effects (font (size 1 1) (thickness 0.15)))
     )
@@
     (tags "capacitor 0805")
     (attr smd)
-    (fp_text reference C4 (at 0 -1.5 90) (layer F.SilkS)
+    (fp_text reference C4 (at 3.5 0 180) (layer F.SilkS)
       (effects (font (size 1 1) (thickness 0.15)))
     )
@@
     (tags "capacitor 0805")
     (attr smd)
-    (fp_text reference C5 (at 0 -1.5 90) (layer F.SilkS)
+    (fp_text reference C5 (at 3.5 0 180) (layer F.SilkS)
       (effects (font (size 1 1) (thickness 0.15)))
     )
@@
     (tags "LED led 0805 SMD smd SMT smt smdled SMDLED smtled SMTLED")
     (attr smd)
-    (fp_text reference D1 (at 0 -1.45 90) (layer F.SilkS)
+    (fp_text reference D1 (at -3 0 180) (layer F.SilkS)
       (effects (font (size 1 1) (thickness 0.15)))
     )
@@
     (tags "LED led 0805 SMD smd SMT smt smdled SMDLED smtled SMTLED")
     (attr smd)
-    (fp_text reference D2 (at 0 -1.45 270) (layer F.SilkS)
+    (fp_text reference D2 (at -2.9 0 360) (layer F.SilkS)
       (effects (font (size 1 1) (thickness 0.15)))
     )
@@
   (module device.farm:Micro-Match-FOB-12 locked placed (layer F.Cu)
     (at 110 135)
-    (fp_text reference DO1 (at 0 5) (layer F.SilkS)
+    (fp_text reference DO1 (at 0 0) (layer F.SilkS)
       (effects (font (size 1 1) (thickness 0.15)))
     )
@@
   (module device.farm:Micro-Match-FOB-4 placed (layer F.Cu)
     (at 110.095 98)
-    (fp_text reference I2C1 (at 0 5) (layer F.SilkS)
+    (fp_text reference I2C1 (at 0 0) (layer F.SilkS)
       (effects (font (size 1 1) (thickness 0.15)))
     )
@@
     (tags "resistor 0805")
     (attr smd)
-    (fp_text reference L1 (at 0 -1.65) (layer F.SilkS)
+    (fp_text reference L1 (at -0.05 2) (layer F.SilkS)
       (effects (font (size 1 1) (thickness 0.15)))
     )
@@
   (module device.farm:DG301-5.0-02 locked placed (layer F.Cu)
     (at 127 136)
-    (fp_text reference MAINS1 (at 0 4.4) (layer F.SilkS)
+    (fp_text reference MAINS1 (at 0.5 -3) (layer F.SilkS)
       (effects (font (size 1 1) (thickness 0.15)))
     )
@@
     (tags "resistor 0805")
     (attr smd)
-    (fp_text reference R1 (at 0 -1.65 270) (layer F.SilkS)
+    (fp_text reference R1 (at -3.55 0 360) (layer F.SilkS)
       (effects (font (size 1 1) (thickness 0.15)))
     )
@@
     (tags "resistor 0805")
     (attr smd)
-    (fp_text reference R3 (at 0 -1.65 270) (layer F.SilkS)
+    (fp_text reference R3 (at 3 0 360) (layer F.SilkS)
       (effects (font (size 1 1) (thickness 0.15)))
     )
@@
     (tags "resistor 0805")
     (attr smd)
-    (fp_text reference R2 (at 0 -1.65 90) (layer F.SilkS)
+    (fp_text reference R2 (at 3.55 -0.05 180) (layer F.SilkS)
       (effects (font (size 1 1) (thickness 0.15)))
     )
@@
     (tags "resistor 0805")
     (attr smd)
-    (fp_text reference R4 (at 0 -1.65 90) (layer F.SilkS)
+    (fp_text reference R4 (at 3 0 180) (layer F.SilkS)
       (effects (font (size 1 1) (thickness 0.15)))
     )
@@
     (tags "resistor 0805")
     (attr smd)
-    (fp_text reference R5 (at 0 -1.65 90) (layer F.SilkS)
+    (fp_text reference R5 (at 2.55 0 180) (layer F.SilkS)
       (effects (font (size 1 1) (thickness 0.15)))
     )
@@
     (tags "resistor 0805")
     (attr smd)
-    (fp_text reference R6 (at 0 -1.65 90) (layer F.SilkS)
+    (fp_text reference R6 (at 2.55 0 180) (layer F.SilkS)
       (effects (font (size 1 1) (thickness 0.15)))
     )
@@
     (tags "resistor 0805")
     (attr smd)
-    (fp_text reference R7 (at 0 -1.65 270) (layer F.SilkS)
+    (fp_text reference R7 (at -2.55 0 360) (layer F.SilkS)
       (effects (font (size 1 1) (thickness 0.15)))
     )
@@
     (tags "resistor 0805")
     (attr smd)
-    (fp_text reference R8 (at 0 -1.65 270) (layer F.SilkS)
+    (fp_text reference R8 (at -2.55 0 360) (layer F.SilkS)
       (effects (font (size 1 1) (thickness 0.15)))
     )
@@
     (tags "resistor 0805")
     (attr smd)
-    (fp_text reference R9 (at 0 -1.65 90) (layer F.SilkS)
+    (fp_text reference R9 (at 2.55 0 180) (layer F.SilkS)
       (effects (font (size 1 1) (thickness 0.15)))
     )
@@
   (module device.farm:DG301-5.0-03 locked placed (layer F.Cu)
     (at 83 136)
-    (fp_text reference TS1 (at 0 4.4) (layer F.SilkS)
+    (fp_text reference TS1 (at 0 -3) (layer F.SilkS)
       (effects (font (size 1 1) (thickness 0.15)))
     )
@@
     (tags SOT-23-5)
     (attr smd)
-    (fp_text reference U2 (at 0 -2.9 180) (layer F.SilkS)
+    (fp_text reference U2 (at 0.1 -2.55 180) (layer F.SilkS)
       (effects (font (size 1 1) (thickness 0.15)))
     )
@@
   (module device.farm:HLK-PM01 locked placed (layer F.Cu)
     (at 129.5 108.3 90)
-    (fp_text reference U3 (at 0 -1.27 90) (layer F.SilkS)
+    (fp_text reference U3 (at 18.3 0 180) (layer F.SilkS)
       (effects (font (size 1 1) (thickness 0.15)))
     )
@@
     (tags "SOIC 1.27")
     (attr smd)
-    (fp_text reference U1 (at 0 -6.25 90) (layer F.SilkS)
+    (fp_text reference U1 (at 0 6.5 90) (layer F.SilkS)
       (effects (font (size 1 1) (thickness 0.15)))
     )
@@
   (module device.farm:ESP-12 placed (layer F.Cu)
     (at 104.5 115.75 90)
-    (fp_text reference U4 (at 4.25 -1 180) (layer F.SilkS)
+    (fp_text reference U4 (at 0.25 1 270) (layer F.SilkS)
       (effects (font (size 1 1) (thickness 0.15)))
     )
@@
   (module device.farm:Micro-Match-FOB-6 placed (layer F.Cu)
     (at 92.825 98)
-    (fp_text reference X1 (at 0 5) (layer F.SilkS)
+    (fp_text reference X1 (at 0.175 0) (layer F.SilkS)
       (effects (font (size 1 1) (thickness 0.15)))
     )
@@
       (rotate (xyz 0 0 0))
     )
+  )
+  (gr_text Address: (at 91.5 117.5 270) (layer B.SilkS)
+    (effects (font (size 1.5 1.5) (thickness 0.3)) (justify mirror))
+  )
+  (gr_line (start 85.5 121.5) (end 85.5 95.5) (layer B.SilkS) (width 10))
+  (gr_text CC-BY-SA (at 128 86.5) (layer F.SilkS)
+    (effects (font (size 1.5 1.5) (thickness 0.3)))
+  )
+  (gr_text "DO6TS1A 1.0" (at 111 86.5) (layer F.SilkS)
+    (effects (font (size 1.5 1.5) (thickness 0.3)))
+  )
+  (gr_text DEVICE.FARM (at 93 86.5) (layer F.SilkS)
+    (effects (font (size 1.5 1.5) (thickness 0.3)))
+  )
+  (gr_text "TTL OUT" (at 110 129.5) (layer F.SilkS)
+    (effects (font (size 1.5 1.5) (thickness 0.3)))
+  )
+  (gr_text I2C (at 116 98) (layer F.SilkS)
+    (effects (font (size 1.5 1.5) (thickness 0.3)))
+  )
+  (gr_text ESPP (at 93 93) (layer F.SilkS)
+    (effects (font (size 1.5 1.5) (thickness 0.3)))
+  )
+  (gr_text 230VAC (at 129.5 130.5) (layer F.SilkS)
+    (effects (font (size 1.5 1.5) (thickness 0.3)))
+  )
+  (gr_text TS:GND/DATA/3V3 (at 91.5 131) (layer F.SilkS)
+    (effects (font (size 1 1) (thickness 0.25)))
   )
   (dimension 30 (width 0.3) (layer Dwgs.User)
@@
   (segment (start 112.635 124.92) (end 105.555 132) (width 0.4) (layer F.Cu) (net 11))
   (segment (start 105.555 132) (end 105.555 132.75) (width 0.4) (layer F.Cu) (net 11))
-  (segment (start 109.245 129.881458) (end 109.245 130.85) (width 0.4) (layer F.Cu) (net 12))
   (segment (start 113.905 123.65) (end 113.905 125.221458) (width 0.4) (layer F.Cu) (net 12))
-  (segment (start 108.095 132) (end 108.095 132.75) (width 0.4) (layer F.Cu) (net 12))
-  (segment (start 113.905 125.221458) (end 109.245 129.881458) (width 0.4) (layer F.Cu) (net 12))
-  (segment (start 109.245 130.85) (end 108.095 132) (width 0.4) (layer F.Cu) (net 12))
-  (segment (start 115.175 124.8) (end 110.635 129.34) (width 0.4) (layer F.Cu) (net 13))
-  (segment (start 115.175 123.65) (end 115.175 124.8) (width 0.4) (layer F.Cu) (net 13))
-  (segment (start 110.635 129.34) (end 110.635 130.85) (width 0.4) (layer F.Cu) (net 13))
+  (segment (start 113.905 125.221458) (end 108.095 131.031458) (width 0.4) (layer F.Cu) (net 12))
+  (segment (start 108.095 131.031458) (end 108.095 132.75) (width 0.4) (layer F.Cu) (net 12))
+  (segment (start 115.175 123.65) (end 115.175 125.512833) (width 0.4) (layer F.Cu) (net 13))
+  (segment (start 115.175 125.512833) (end 110.635 130.052833) (width 0.4) (layer F.Cu) (net 13))
+  (segment (start 110.635 130.052833) (end 110.635 130.85) (width 0.4) (layer F.Cu) (net 13))
   (segment (start 110.635 130.85) (end 110.635 132.75) (width 0.4) (layer F.Cu) (net 13))
   (segment (start 118.5 126.675) (end 113.175 132) (width 0.4) (layer F.Cu) (net 14))
