File: board/DO6TS1A.kicad_pcb (KiCad board)
At the start: 2 copper layers, 60 x 55 mm, 29 parts, among them U1 PCF8574, U2 RT9193, U3 HLK-PM01, U4 ESP-12, X1 ESP-PROG

Commit message: WIP
Parts:
- added C8: 100n, Capacitors_SMD:C_1210, B.Cu at (132.0, 113.5)
- added C9: 1u, Capacitors_SMD:C_0805, B.Cu at (122.0, 98.0)
- added R10: 1k5, Resistors_SMD:R_1206, B.Cu at (133.5, 109.0)
- added R11: 1k5, Resistors_SMD:R_0805, B.Cu at (129.0, 98.0)
- added R12: 56k, Resistors_SMD:R_0805, B.Cu at (125.5, 98.0)
- added TARIFF1: Conn_01x02, device.farm:DG301-5.0-02, F.Cu at (119.5, 136.0)
- added U5: LTV-354T, Housings_SOIC:SO-4_4.4x3.6mm_Pitch2.54mm, B.Cu at (133.5, 101.5)
- moved D3 15.1 mm to (101.5, 98.5), turned to 270 degrees
- moved DO1 3.91 mm to (106.1, 135.0)
- moved MAINS1 2.50 mm to (129.5, 136.0)
Connections:
- D3 pad 1: /ESP/5V-PROG -> Net-(C3-Pad1)
- D3 pad 2: /ESP/5V-MAINS -> /ESP/3V3-PROG
- D3 pad 3: /5V -> Net-(D3-Pad3)
- I2C1 pad 4: /5V -> VCC
- L1 pad 2: Net-(C3-Pad1) -> Net-(D3-Pad3)
- U3 pad 4: /ESP/5V-MAINS -> /5V
- U4 pad 14: (no net) -> /TARIFF
- X1 pad 6: /ESP/5V-PROG -> /ESP/3V3-PROG
Routing:
- net VCC: track 112.3 -> 154.7 mm, vias 0 -> 6
- net /TARIFF: track 0.00 -> 40.4 mm, vias 0 -> 1
- net Net-(TARIFF1-Pad1): track 0.00 -> 37.4 mm, vias 0 -> 1
- net /ESP/5V-PROG: track 33.4 -> 0.00 mm, vias 2 -> 0
- net Net-(C8-Pad2): track 0.00 -> 29.0 mm
- net /ESP/5V-MAINS: track 24.1 -> 0.00 mm
- net /5V: track 78.4 -> 99.2 mm
- net /ESP/3V3-PROG: track 0.00 -> 6.13 mm
- net Net-(C3-Pad1): track 6.46 -> 11.3 mm
- net Net-(D3-Pad3): track 0.00 -> 4.71 mm
- net Net-(R10-Pad1): track 0.00 -> 4.42 mm
- net Net-(DO1-Pad1): track 12.6 -> 17.0 mm
- net Net-(DO1-Pad3): track 12.0 -> 15.6 mm
- net Net-(DO1-Pad9): track 21.5 -> 24.7 mm
- net Net-(C8-Pad1): track 0.00 -> 3.02 mm
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Other:
- board text added: "MAINS"
- board text added: "TARIFF"

Commit message: WIP
Parts:
- C1, C2, C3, C4, C5, C6, C7, C9: footprint Capacitors_SMD:C_0805 -> Capacitor_SMD:C_0805_2012Metric
- C8: footprint Capacitors_SMD:C_1210 -> Capacitor_SMD:C_1210_3225Metric
- D1, D2: footprint LEDs:LED_0805 -> LED_SMD:LED_0805_2012Metric
- D3: footprint TO_SOT_Packages_SMD:SOT-23 -> Package_TO_SOT_SMD:SOT-23
- DO1: footprint device.farm:Micro-Match-FOB-12 -> Drake:Micro-Match-FOB-12
- I2C1: footprint device.farm:Micro-Match-FOB-4 -> Drake:Micro-Match-FOB-4
- L1, R1, R11, R12, R2, R3, R4, R5, R6, R7, R8, R9: footprint Resistors_SMD:R_0805 -> Resistor_SMD:R_0805_2012Metric
- MAINS1, TARIFF1: footprint device.farm:DG301-5.0-02 -> Drake:DG301-5.0-02
- R10: footprint Resistors_SMD:R_1206 -> Resistor_SMD:R_1206_3216Metric
- TS1: footprint device.farm:DG301-5.0-03 -> Drake:DG301-5.0-03
- U1: footprint Housings_SOIC:SOIC-16W_7.5x10.3mm_Pitch1.27mm -> Package_SO:SOIC-16W_7.5x10.3mm_P1.27mm
- U3: footprint device.farm:HLK-PM01 -> Drake:HLK-PM01
- U4: footprint device.farm:ESP-12 -> Drake:ESP-12
- U5: footprint Housings_SOIC:SO-4_4.4x3.6mm_Pitch2.54mm -> Package_SO:SO-4_4.4x3.6mm_P2.54mm
- X1: footprint device.farm:Micro-Match-FOB-6 -> Drake:Micro-Match-FOB-6
Connections:
- U1 pad 13: (no net) -> Net-(U1-Pad13)
- U4 pad 2: (no net) -> /ESP/ADC
- U4 pad 4: (no net) -> /ESP/GPIO16
- U4 pad 7: (no net) -> /ESP/GPIO13
Routing:
- net /SDA: track 47.5 -> 48.4 mm
- net Net-(DO1-Pad5): track 14.2 -> 14.8 mm
Other:
- board text added: "Drake"
- board text removed: "DEVICE.FARM"

Commit message: WIP
Parts:
- U2: footprint TO_SOT_Packages_SMD:SOT-23-5 -> Package_TO_SOT_SMD:SOT-23-5
Connections:
- U1 pad 13: Net-(U1-Pad13) -> unconnected-(U1-Pad13)
Other:
- net class Default removed
