File: board/DO6TS1A.sch (KiCad schematic (older format))
At the start: 11 parts, among them U3 PCF8574

Commit message: WIP
Parts:
- renumbered D2 to D1, D3 to D2, R3 to R2, R2 to R3, U3 to U1
Changed lines of the file:
@@
 $EndDescr
 $Comp
-L R R2
+L R R3
 U 1 1 5762449B
 P 8300 4250
-F 0 "R2" V 8500 4250 50  0000 C CNN
+F 0 "R3" V 8500 4250 50  0000 C CNN
 F 1 "270R" V 8400 4250 50  0000 C CNN
 F 2 "Resistors_SMD:R_0805" V 8230 4250 50  0001 C CNN
@@
 $EndComp
 $Comp
-L LED D2
+L LED D1
 U 1 1 57624710
 P 8000 4250
-F 0 "D2" H 8000 4050 50  0000 C CNN
+F 0 "D1" H 8000 4050 50  0000 C CNN
 F 1 "LED" H 8000 4150 50  0000 C CNN
 F 2 "LEDs:LED_0805" H 8000 4250 50  0001 C CNN
@@
 3V3
 $Comp
-L PCF8574 U3
+L PCF8574 U1
 U 1 1 5A97FD34
 P 7100 3550
-F 0 "U3" H 6750 4150 50  0000 L CNN
+F 0 "U1" H 6750 4150 50  0000 L CNN
 F 1 "PCF8574" H 7200 4150 50  0000 L CNN
 F 2 "Housings_SOIC:SOIC-16W_7.5x10.3mm_Pitch1.27mm" H 7100 3550 50  0001 C CNN
@@
 $EndComp
 $Comp
-L LED D3
+L LED D2
 U 1 1 5A9805A6
 P 8000 4600
-F 0 "D3" H 8000 4400 50  0000 C CNN
+F 0 "D2" H 8000 4400 50  0000 C CNN
 F 1 "LED" H 8000 4500 50  0000 C CNN
 F 2 "LEDs:LED_0805" H 8000 4600 50  0001 C CNN
@@
 $EndComp
 $Comp
-L VCC #PWR01
+L VCC #PWR5
 U 1 1 5A980AF9
 P 7100 2850
-F 0 "#PWR01" H 7100 2700 50  0001 C CNN
+F 0 "#PWR5" H 7100 2700 50  0001 C CNN
 F 1 "VCC" H 7100 3000 50  0000 C CNN
 F 2 "" H 7100 2850 50  0001 C CNN
@@
 $EndComp
 $Comp
-L VCC #PWR02
+L VCC #PWR8
 U 1 1 5A980B68
 P 8600 4150
-F 0 "#PWR02" H 8600 4000 50  0001 C CNN
+F 0 "#PWR8" H 8600 4000 50  0001 C CNN
 F 1 "VCC" H 8600 4300 50  0000 C CNN
 F 2 "" H 8600 4150 50  0001 C CNN
@@
 $EndComp
 $Comp
-L GND #PWR03
+L GND #PWR6
 U 1 1 5A980CE2
 P 7100 4250
-F 0 "#PWR03" H 7100 4000 50  0001 C CNN
+F 0 "#PWR6" H 7100 4000 50  0001 C CNN
 F 1 "GND" H 7100 4100 50  0000 C CNN
 F 2 "" H 7100 4250 50  0001 C CNN
@@
 $EndComp
 $Comp
-L R R3
+L R R2
 U 1 1 5A981B02
 P 5300 3350
-F 0 "R3" V 5500 3350 50  0000 C CNN
+F 0 "R2" V 5500 3350 50  0000 C CNN
 F 1 "10k" V 5400 3350 50  0000 C CNN
 F 2 "Resistors_SMD:R_0805" V 5230 3350 50  0001 C CNN
@@
 	5300 3150 5300 3200
 $Comp
-L VCC #PWR04
+L VCC #PWR1
 U 1 1 5A98213D
 P 5250 3100
-F 0 "#PWR04" H 5250 2950 50  0001 C CNN
+F 0 "#PWR1" H 5250 2950 50  0001 C CNN
 F 1 "VCC" H 5250 3250 50  0000 C CNN
 F 2 "" H 5250 3100 50  0001 C CNN
@@
 $EndComp
 $Comp
-L GND #PWR05
+L GND #PWR3
 U 1 1 5A98297A
 P 5700 2300
-F 0 "#PWR05" H 5700 2050 50  0001 C CNN
+F 0 "#PWR3" H 5700 2050 50  0001 C CNN
 F 1 "GND" H 5700 2150 50  0000 C CNN
 F 2 "" H 5700 2300 50  0001 C CNN
@@
 $EndComp
 $Comp
-L VCC #PWR06
+L VCC #PWR2
 U 1 1 5A982A5B
 P 5700 2100
-F 0 "#PWR06" H 5700 1950 50  0001 C CNN
+F 0 "#PWR2" H 5700 1950 50  0001 C CNN
 F 1 "VCC" H 5700 2250 50  0000 C CNN
 F 2 "" H 5700 2100 50  0001 C CNN
@@
 5V
 $Comp
-L GND #PWR07
+L GND #PWR7
 U 1 1 5A983E03
 P 7550 2300
-F 0 "#PWR07" H 7550 2050 50  0001 C CNN
+F 0 "#PWR7" H 7550 2050 50  0001 C CNN
 F 1 "GND" H 7550 2150 50  0000 C CNN
 F 2 "" H 7550 2300 50  0001 C CNN
@@
 $EndComp
 $Comp
-L GND #PWR08
+L GND #PWR4
 U 1 1 5A98400C
 P 6400 3700
-F 0 "#PWR08" H 6400 3450 50  0001 C CNN
+F 0 "#PWR4" H 6400 3450 50  0001 C CNN
 F 1 "GND" H 6400 3550 50  0000 C CNN
 F 2 "" H 6400 3700 50  0001 C CNN

Commit message: WIP
Parts:
- added C8: 100n, Capacitors_SMD:C_1210, symbol C
- added C9: 1u, Capacitors_SMD:C_0805, symbol C
- added R10: 1k5, Resistors_SMD:R_1206, symbol R
- added R11: 1k5, Resistors_SMD:R_0805, symbol R
- added R12: 56k, Resistors_SMD:R_0805, symbol R
- added TARIFF1: Conn_01x02, device.farm:DG301-5.0-02, symbol Conn_01x02
- added U5: LTV-354T, Housings_SOIC:SO-4_4.4x3.6mm_Pitch2.54mm, symbol LTV-354T
Connections:
- net labels added: TARIFF
- wire segments 37 -> 46
- no-connect marks 5 -> 4
Other:
- note added: "http://tinyurl.com/y9cn5mc4"
- note added: "http://tinyurl.com/y9xpjohp"
