File: board/esp-mains.sch (KiCad schematic (older format))
At the start: 18 parts, among them U1 RT9193, U2 HLK-PM01, U4 ESP-12, X1 ESP-PROG

Commit message: WIP
Parts:
- C3: value 47u -> 1u
- renumbered C8 to C4, C9 to C5, C4 to C6, D1 to D3, U1 to U2, U2 to U3
Connections:
- wire segments 31 -> 30
Changed lines of the file:
@@
 $EndComp
 $Comp
-L HLK-PM01 U2
+L HLK-PM01 U3
 U 1 1 5777B23B
 P 4050 2200
-F 0 "U2" H 4050 2637 60  0000 C CNN
+F 0 "U3" H 4050 2637 60  0000 C CNN
 F 1 "HLK-PM01" H 4050 2531 60  0000 C CNN
 F 2 "device.farm:HLK-PM01" H 4050 2200 60  0001 C CNN
@@
 $EndComp
 $Comp
-L GND #PWR09
+L GND #PWR15
 U 1 1 5777B23D
 P 4550 2350
-F 0 "#PWR09" H 4550 2100 50  0001 C CNN
+F 0 "#PWR15" H 4550 2100 50  0001 C CNN
 F 1 "GND" V 4555 2222 50  0000 R CNN
 F 2 "" H 4550 2350 50  0000 C CNN
@@
 $EndComp
 $Comp
-L GND #PWR010
+L GND #PWR12
 U 1 1 5777B244
 P 3450 5400
-F 0 "#PWR010" H 3450 5150 50  0001 C CNN
+F 0 "#PWR12" H 3450 5150 50  0001 C CNN
 F 1 "GND" H 3455 5227 50  0000 C CNN
 F 2 "" H 3450 5400 50  0000 C CNN
@@
 $EndComp
 $Comp
-L GND #PWR011
+L GND #PWR13
 U 1 1 5777B245
 P 3900 5400
-F 0 "#PWR011" H 3900 5150 50  0001 C CNN
+F 0 "#PWR13" H 3900 5150 50  0001 C CNN
 F 1 "GND" H 3905 5227 50  0000 C CNN
 F 2 "" H 3900 5400 50  0000 C CNN
@@
 $EndComp
 $Comp
-L RT9193 U1
+L RT9193 U2
 U 1 1 5777B246
 P 3450 4950
-F 0 "U1" H 3450 5387 60  0000 C CNN
+F 0 "U2" H 3450 5387 60  0000 C CNN
 F 1 "RT9193" H 3450 5281 60  0000 C CNN
 F 2 "TO_SOT_Packages_SMD:SOT-23-5" H 3450 4950 60  0001 C CNN
@@
 $EndComp
 $Comp
-L GND #PWR012
+L GND #PWR11
 U 1 1 5777B247
 P 2600 5400
-F 0 "#PWR012" H 2600 5150 50  0001 C CNN
+F 0 "#PWR11" H 2600 5150 50  0001 C CNN
 F 1 "GND" H 2605 5227 50  0000 C CNN
 F 2 "" H 2600 5400 50  0000 C CNN
@@
 P 4300 5050
 F 0 "C3" H 4415 5096 50  0000 L CNN
-F 1 "47u" H 4415 5005 50  0000 L CNN
+F 1 "1u" H 4415 5005 50  0000 L CNN
 F 2 "Capacitors_SMD:C_0805" H 4338 4900 50  0001 C CNN
 F 3 "" H 4300 5050 50  0000 C CNN
@@
 $EndComp
 $Comp
-L GND #PWR013
+L GND #PWR14
 U 1 1 5777B249
 P 4300 5400
-F 0 "#PWR013" H 4300 5150 50  0001 C CNN
+F 0 "#PWR14" H 4300 5150 50  0001 C CNN
 F 1 "GND" H 4305 5227 50  0000 C CNN
 F 2 "" H 4300 5400 50  0000 C CNN
@@
 5V
 $Comp
-L C C4
+L C C6
 U 1 1 5777B24E
-P 4900 5050
-F 0 "C4" H 5015 5096 50  0000 L CNN
-F 1 "100n" H 5015 5005 50  0000 L CNN
-F 2 "Capacitors_SMD:C_0805" H 4938 4900 50  0001 C CNN
-F 3 "" H 4900 5050 50  0000 C CNN
-	1    4900 5050
-	1    0    0    -1
-$EndComp
-$Comp
-L GND #PWR014
-U 1 1 5777B24F
-P 4900 5400
-F 0 "#PWR014" H 4900 5150 50  0001 C CNN
-F 1 "GND" H 4905 5227 50  0000 C CNN
-F 2 "" H 4900 5400 50  0000 C CNN
-F 3 "" H 4900 5400 50  0000 C CNN
-	1    4900 5400
+P 6400 5400
+F 0 "C6" H 6400 5500 50  0000 L CNN
+F 1 "100n" H 6400 5300 50  0000 L CNN
+F 2 "Capacitors_SMD:C_0805" H 6438 5250 50  0001 C CNN
+F 3 "" H 6400 5400 50  0000 C CNN
+	1    6400 5400
 	1    0    0    -1
 $EndComp
@@
 RESET
 $Comp
-L GND #PWR015
+L GND #PWR20
 U 1 1 5777B25A
 P 7550 5200
-F 0 "#PWR015" H 7550 4950 50  0001 C CNN
+F 0 "#PWR20" H 7550 4950 50  0001 C CNN
 F 1 "GND" H 7555 5027 50  0000 C CNN
 F 2 "" H 7550 5200 50  0000 C CNN
@@
 $EndComp
 $Comp
-L GND #PWR016
+L GND #PWR22
 U 1 1 5777B260
 P 9700 5500
-F 0 "#PWR016" H 9700 5250 50  0001 C CNN
+F 0 "#PWR22" H 9700 5250 50  0001 C CNN
 F 1 "GND" H 9705 5327 50  0000 C CNN
 F 2 "" H 9700 5500 50  0000 C CNN
@@
 $EndComp
 $Comp
-L GND #PWR017
+L GND #PWR21
 U 1 1 5777B262
 P 9700 5200
-F 0 "#PWR017" H 9700 4950 50  0001 C CNN
+F 0 "#PWR21" H 9700 4950 50  0001 C CNN
 F 1 "GND" H 9705 5027 50  0000 C CNN
 F 2 "" H 9700 5200 50  0000 C CNN
@@
 $EndComp
 $Comp
-L VCC #PWR018
+L VCC #PWR23
 U 1 1 5777BAC2
 P 9800 4400
-F 0 "#PWR018" H 9800 4250 50  0001 C CNN
+F 0 "#PWR23" H 9800 4250 50  0001 C CNN
 F 1 "VCC" V 9817 4528 50  0000 L CNN
 F 2 "" H 9800 4400 50  0000 C CNN
@@
 $EndComp
 $Comp
-L VCC #PWR019
+L VCC #PWR17
 U 1 1 5777C817
-P 6050 5200
-F 0 "#PWR019" H 6050 5050 50  0001 C CNN
-F 1 "VCC" V 6068 5327 50  0000 L CNN
-F 2 "" H 6050 5200 50  0000 C CNN
-F 3 "" H 6050 5200 50  0000 C CNN
-	1    6050 5200
-	0    -1   -1   0
-$EndComp
-$Comp
-L VCC #PWR020
+P 5900 5200
+F 0 "#PWR17" H 5900 5050 50  0001 C CNN
+F 1 "VCC" V 5918 5327 50  0000 L CNN
+F 2 "" H 5900 5200 50  0000 C CNN
+F 3 "" H 5900 5200 50  0000 C CNN
+	1    5900 5200
+	0    -1   -1   0
+$EndComp
+$Comp
+L VCC #PWR16
 U 1 1 5777D0FB
-P 5050 4800
-F 0 "#PWR020" H 5050 4650 50  0001 C CNN
-F 1 "VCC" V 5067 4928 50  0000 L CNN
-F 2 "" H 5050 4800 50  0000 C CNN
-F 3 "" H 5050 4800 50  0000 C CNN
-	1    5050 4800
+P 4950 4800
+F 0 "#PWR16" H 4950 4650 50  0001 C CNN
+F 1 "VCC" V 4967 4928 50  0000 L CNN
+F 2 "" H 4950 4800 50  0000 C CNN
+F 3 "" H 4950 4800 50  0000 C CNN
+	1    4950 4800
 	0    1    1    0
 $EndComp
@@
 GPIO5
 $Comp
-L GND #PWR021
+L GND #PWR10
 U 1 1 5778ED26
 P 1850 2300
-F 0 "#PWR021" H 1850 2050 50  0001 C CNN
+F 0 "#PWR10" H 1850 2050 50  0001 C CNN
 F 1 "GND" V 1855 2127 50  0000 C CNN
 F 2 "" H 1850 2300 50  0000 C CNN
@@
 $EndComp
 $Comp
-L PWR_FLAG #FLG022
+L PWR_FLAG #FLG2
 U 1 1 5778ED65
 P 1850 2300
-F 0 "#FLG022" H 1850 2395 50  0001 C CNN
+F 0 "#FLG2" H 1850 2395 50  0001 C CNN
 F 1 "PWR_FLAG" V 1850 2650 50  0000 C CNN
 F 2 "" H 1850 2300 50  0000 C CNN
@@
 $EndComp
 $Comp
-L VCC #PWR023
+L VCC #PWR9
 U 1 1 57790C33
 P 1850 2100
-F 0 "#PWR023" H 1850 1950 50  0001 C CNN
+F 0 "#PWR9" H 1850 1950 50  0001 C CNN
 F 1 "VCC" V 1868 2227 50  0000 L CNN
 F 2 "" H 1850 2100 50  0000 C CNN
@@
 $EndComp
 $Comp
-L PWR_FLAG #FLG024
+L PWR_FLAG #FLG1
 U 1 1 57790FA9
 P 1850 2100
-F 0 "#FLG024" H 1850 2195 50  0001 C CNN
+F 0 "#FLG1" H 1850 2195 50  0001 C CNN
 F 1 "PWR_FLAG" V 1850 2450 50  0000 C CNN
 F 2 "" H 1850 2100 50  0000 C CNN
@@
 $EndComp
 $Comp
-L D_Schottky_x2_KCom_AAK D1
+L D_Schottky_x2_KCom_AAK D3
 U 1 1 579135F5
 P 2200 4800
-F 0 "D1" V 2246 4880 50  0000 L CNN
+F 0 "D3" V 2246 4880 50  0000 L CNN
 F 1 "BAT54C" V 2155 4880 50  0000 L CNN
 F 2 "TO_SOT_Packages_SMD:SOT-23" H 2200 4800 50  0001 C CNN
@@
 Text HLabel 2600 4700 1    60   Output ~ 0
 5V
-Text HLabel 5100 4600 2    60   Output ~ 0
+Text HLabel 5000 4600 2    60   Output ~ 0
 3V3
 Wire Wire Line
@@
 	4300 4900 4300 4800
 Connection ~ 4300 4800
-Wire Wire Line
-	4900 4900 4900 4800
-Connection ~ 4900 4800
-Wire Wire Line
-	4900 5400 4900 5200
 Wire Wire Line
 	9750 5000 9700 5000
@@
 	3900 4800 4450 4800
 Wire Wire Line
-	4750 4800 5050 4800
-Wire Wire Line
-	5100 4600 5000 4600
-Wire Wire Line
-	5000 4600 5000 4800
-Connection ~ 5000 4800
-$Comp
-L C C9
+	4750 4800 4950 4800
+Wire Wire Line
+	5000 4600 4900 4600
+Wire Wire Line
+	4900 4600 4900 4800
+Connection ~ 4900 4800
+$Comp
+L C C5
 U 1 1 5A74BDF9
-P 6350 5400
-F 0 "C9" H 6500 5450 50  0000 L CNN
-F 1 "47u" H 6465 5355 50  0000 L CNN
-F 2 "Capacitors_SMD:C_0805" H 6388 5250 50  0001 C CNN
-F 3 "" H 6350 5400 50  0000 C CNN
-	1    6350 5400
-	1    0    0    -1
-$EndComp
-$Comp
-L C C8
+P 6200 5400
+F 0 "C5" H 6200 5500 50  0000 L CNN
+F 1 "47u" H 6200 5300 50  0000 L CNN
+F 2 "Capacitors_SMD:C_0805" H 6238 5250 50  0001 C CNN
+F 3 "" H 6200 5400 50  0000 C CNN
+	1    6200 5400
+	1    0    0    -1
+$EndComp
+$Comp
+L C C4
 U 1 1 5A74BEDA
-P 6150 5400
-F 0 "C8" H 5950 5450 50  0000 L CNN
-F 1 "47u" H 5900 5350 50  0000 L CNN
-F 2 "Capacitors_SMD:C_0805" H 6188 5250 50  0001 C CNN
-F 3 "" H 6150 5400 50  0000 C CNN
-	1    6150 5400
-	1    0    0    -1
-$EndComp
-$Comp
-L GND #PWR025
+P 6000 5400
+F 0 "C4" H 6000 5500 50  0000 L CNN
+F 1 "47u" H 6000 5300 50  0000 L CNN
+F 2 "Capacitors_SMD:C_0805" H 6038 5250 50  0001 C CNN
+F 3 "" H 6000 5400 50  0000 C CNN
+	1    6000 5400
+	1    0    0    -1
+$EndComp
+$Comp
+L GND #PWR18
 U 1 1 5A74BFA4
-P 6250 5650
-F 0 "#PWR025" H 6250 5400 50  0001 C CNN
-F 1 "GND" H 6255 5477 50  0000 C CNN
-F 2 "" H 6250 5650 50  0000 C CNN
-F 3 "" H 6250 5650 50  0000 C CNN
-	1    6250 5650
-	1    0    0    -1
-$EndComp
-Wire Wire Line
-	6050 5200 6450 5200
-Wire Wire Line
-	6350 5250 6350 5200
-Connection ~ 6350 5200
-Wire Wire Line
-	6150 5250 6150 5200
-Connection ~ 6150 5200
-Wire Wire Line
-	6250 5650 6250 5550
-Wire Wire Line
-	6150 5550 6350 5550
-Connection ~ 6250 5550
+P 6200 5650
+F 0 "#PWR18" H 6200 5400 50  0001 C CNN
+F 1 "GND" H 6205 5477 50  0000 C CNN
+F 2 "" H 6200 5650 50  0000 C CNN
+F 3 "" H 6200 5650 50  0000 C CNN
+	1    6200 5650
+	1    0    0    -1
+$EndComp
+Wire Wire Line
+	5900 5200 6450 5200
+Wire Wire Line
+	6200 5250 6200 5200
+Connection ~ 6200 5200
+Wire Wire Line
+	6000 5250 6000 5200
+Connection ~ 6000 5200
+Wire Wire Line
+	6000 5550 6400 5550
 $Comp
 L ESP-PROG X1
@@
 TX
 $Comp
-L GND #PWR026
+L GND #PWR19
 U 1 1 5A97EADF
 P 7450 3150
-F 0 "#PWR026" H 7450 2900 50  0001 C CNN
+F 0 "#PWR19" H 7450 2900 50  0001 C CNN
 F 1 "GND" H 7455 2977 50  0000 C CNN
 F 2 "" H 7450 3150 50  0000 C CNN
@@
 Text Label 7450 2550 0    60   ~ 0
 5V-PROG
+Wire Wire Line
+	6400 5250 6400 5200
+Connection ~ 6400 5200
+Connection ~ 6200 5550
+Wire Wire Line
+	6200 5650 6200 5550
 $EndSCHEMATC

Commit message: WIP
Connections:
- net labels added: 3V3-PROG
- net labels removed: 5V-PROG
- wire segments 30 -> 29

Commit message: WIP
Parts:
- X1: symbol ESP-PROG -> ESP-PROG-RESCUE-DO6TS1A
Changed lines of the file:
@@
 EESchema Schematic File Version 2
+LIBS:DO6TS1A-rescue
 LIBS:power
 LIBS:device
@@
 	6550 5450 6950 5450
 $Comp
-L ESP-PROG X1
+L ESP-PROG-RESCUE-DO6TS1A X1
 U 1 1 5A97E79C
 P 7000 2850
