File: board/esp-mains.kicad_sch (KiCad schematic)
At the start: 18 parts, among them U2 RT9193, U3 HLK-PM01, U4 ESP-12, X1 ESP-PROG

Commit message: WIP
Parts:
- ?: renamed from U4; value ESP-12 -> (none); footprint Drake:ESP-12 -> (none)
- ?: renamed from U3; value HLK-PM01 -> (none); footprint Drake:HLK-PM01 -> (none)
- ?: renamed from C1; value 1u -> (none); footprint Capacitor_SMD:C_0805_2012Metric -> (none)
- ?: renamed from C2; value 22n -> (none); footprint Capacitor_SMD:C_0805_2012Metric -> (none)
- ?: renamed from U2; value RT9193 -> (none); footprint Package_TO_SOT_SMD:SOT-23-5 -> (none)
- ?: renamed from C3; value 1u -> (none); footprint Capacitor_SMD:C_0805_2012Metric -> (none)
- ?: renamed from C6; value 100n -> (none); footprint Capacitor_SMD:C_0805_2012Metric -> (none)
- ?: renamed from R5; value 10k -> (none); footprint Resistor_SMD:R_0805_2012Metric -> (none)
- ?: renamed from R6; value 10k -> (none); footprint Resistor_SMD:R_0805_2012Metric -> (none)
- ?: renamed from R7; value 10k -> (none); footprint Resistor_SMD:R_0805_2012Metric -> (none)
- ?: renamed from R8; value 10k -> (none); footprint Resistor_SMD:R_0805_2012Metric -> (none)
- ?: renamed from R9; value 10k -> (none); footprint Resistor_SMD:R_0805_2012Metric -> (none)
- ?: renamed from C7; value 100n -> (none); footprint Capacitor_SMD:C_0805_2012Metric -> (none)
- ?: renamed from L1; value Ferrite bead -> (none); footprint Resistor_SMD:R_0805_2012Metric -> (none)
- ?: renamed from D3; value BAT54C -> (none); footprint Package_TO_SOT_SMD:SOT-23 -> (none)
- ?: renamed from C5; value 47u -> (none); footprint Capacitor_SMD:C_0805_2012Metric -> (none)
- ?: renamed from C4; value 47u -> (none); footprint Capacitor_SMD:C_0805_2012Metric -> (none)
- ?: renamed from X1; value ESP-PROG -> (none); footprint Drake:Micro-Match-FOB-6 -> (none)
