File: board/DO6TS1A.kicad_sch (KiCad schematic)
At the start: 18 parts, among them U1 PCF8574, U5 LTV-354T

Commit message: WIP
Parts:
- ?: renamed from R3; value 270R -> (none); footprint Resistor_SMD:R_0805_2012Metric -> (none)
- ?: renamed from D1; value LED -> (none); footprint LED_SMD:LED_0805_2012Metric -> (none)
- ?: renamed from U1; value PCF8574 -> (none); footprint Package_SO:SOIC-16W_7.5x10.3mm_P1.27mm -> (none)
- ?: renamed from DO1; value Conn_02x06_Odd_Even -> (none); footprint Drake:Micro-Match-FOB-12 -> (none)
- ?: renamed from D2; value LED -> (none); footprint LED_SMD:LED_0805_2012Metric -> (none)
- ?: renamed from R4; value 270R -> (none); footprint Resistor_SMD:R_0805_2012Metric -> (none)
- ?: renamed from R1; value 10k -> (none); footprint Resistor_SMD:R_0805_2012Metric -> (none)
- ?: renamed from R2; value 10k -> (none); footprint Resistor_SMD:R_0805_2012Metric -> (none)
- ?: renamed from TS1; value Conn_01x03 -> (none); footprint Drake:DG301-5.0-03 -> (none)
- ?: renamed from I2C1; value I2C -> (none); footprint Drake:Micro-Match-FOB-4 -> (none)
- ?: renamed from MAINS1; value Conn_01x02 -> (none); footprint Drake:DG301-5.0-02 -> (none)
- ?: renamed from U5; value LTV-354T -> (none); footprint Package_SO:SO-4_4.4x3.6mm_P2.54mm -> (none)
- ?: renamed from TARIFF1; value Conn_01x02 -> (none); footprint Drake:DG301-5.0-02 -> (none)
- ?: renamed from C8; value 100n -> (none); footprint Capacitor_SMD:C_1210_3225Metric -> (none)
- ?: renamed from R10; value 1k5 -> (none); footprint Resistor_SMD:R_1206_3216Metric -> (none)
- ?: renamed from R11; value 1k5 -> (none); footprint Resistor_SMD:R_0805_2012Metric -> (none)
- ?: renamed from C9; value 1u -> (none); footprint Capacitor_SMD:C_0805_2012Metric -> (none)
- ?: renamed from R12; value 56k -> (none); footprint Resistor_SMD:R_0805_2012Metric -> (none)

Commit message: WIP
Parts:
- removed ?: (no value), symbol Interface_Expansion:PCF8574
- removed ?: (no value), symbol Device:LED
- removed ?: (no value), symbol Device:R
- removed ?: (no value), symbol Connector_Generic:Conn_01x03
- added C1, C2: 10u, Capacitor_SMD:C_0805_2012Metric, symbol Device:C
- added C10, C11, C12, C13, C14, C15, C16, C17, C18, C19, C20, C21, C22, C8, C9: 100n, Capacitor_SMD:C_0805_2012Metric, symbol Device:C
- added C2, C3: 47u, Capacitor_SMD:C_0805_2012Metric, symbol Device:C
- added C7: 1u, Capacitor_SMD:C_0805_2012Metric, symbol Device:C
- added H1 (x4): MountingHole, MountingHole:MountingHole_3.7mm_Pad_Via, symbol Mechanical:MountingHole
- added J12: PROG, Connector_PinHeader_2.54mm:PinHeader_1x03_P2.54mm_Vertical, symbol Connector_Generic:Conn_01x03
- added R10, R11, R12, R13, R14, R15, R16, R5, R6, R7, R8, R9: 1k5, Resistor_SMD:R_0805_2012Metric, symbol Device:R
- added R17, R18, R19, R20, R21, R22: 100k, Resistor_SMD:R_0805_2012Metric, symbol Device:R
- added R23, R24, R25, R26, R27, R28: 56k, Resistor_SMD:R_0805_2012Metric, symbol Device:R
- added R5: 10k, Resistor_SMD:R_0805_2012Metric, symbol Device:R
- added U1: LM1117MP-3.3, Package_TO_SOT_SMD:SOT-223-3_TabPin2, symbol Regulator_Linear:LM1117MP-3.3
- added U1: YS-12V450A, Drake:YS-12V450A, symbol Drake:PSU
- added U3: ESP32-C3-WROOM-02, Espressif:ESP32-C3-WROOM-02, symbol Espressif:ESP32-C3-WROOM-02
- added U5, U6, U7: LM358, Package_SO:SOIC-8_3.9x4.9mm_P1.27mm, symbol Amplifier_Operational:LM358
- C4: renamed from ?; value (none) -> 100n; footprint (none) -> Capacitor_SMD:C_1210_3225Metric
- C6: renamed from ?; value (none) -> 1u; footprint (none) -> Capacitor_SMD:C_0805_2012Metric
- D1: renamed from ?; value (none) -> LED; footprint (none) -> LED_SMD:LED_0805_2012Metric
- DO1: renamed from ?; value (none) -> Regulators; footprint (none) -> Drake:Micro-Match-FOB-12
- I2C1: renamed from ?; value (none) -> I2C; footprint (none) -> Drake:Micro-Match-FOB-4
- R2: renamed from ?; value (none) -> 1k5; footprint (none) -> Resistor_SMD:R_1206_3216Metric
- R29, R30: renamed from ?; value (none) -> 10k; footprint (none) -> Resistor_SMD:R_0805_2012Metric
- R3: renamed from ?; value (none) -> 1k5; footprint (none) -> Resistor_SMD:R_0805_2012Metric
- R31: renamed from ?; value (none) -> 270R; footprint (none) -> Resistor_SMD:R_0805_2012Metric
- R4: renamed from ?; value (none) -> 56k; footprint (none) -> Resistor_SMD:R_0805_2012Metric
- U2: renamed from ?; value (none) -> LTV-354T; footprint (none) -> Package_SO:SO-4_4.4x3.6mm_P2.54mm
- X1: renamed from ?; value (none) -> MAINS; footprint (none) -> Drake:DG301-5.0-02
- X2: renamed from ?; value (none) -> TARIFF; footprint (none) -> Drake:DG301-5.0-02
Connections:
- net GND: now also D1.1 (K), DO1.1 (Pin_1), DO1.11 (Pin_11), DO1.3 (Pin_3), DO1.5 (Pin_5), DO1.7 (Pin_7), DO1.9 (Pin_9), C1.2, C10.2, C11.2, C12.2, C13.2, C14.2, C15.2, C16.2, C17.2, C18.2, C19.2, C2.2, C2.2, C20.2, C21.2, C22.2, C3.2, C7.1, C8.2, C9.2, J12.2 (Pin_2), R17.2, R18.2, R19.2, R20.2, R21.2, R22.2, U1.1 (GND), U1.3 (OUT-), U3.19 (GND), U3.9 (GND), U5.4 (V-), U6.4 (V-), U7.4 (V-)
- net SCL: now also U3.7 (GPIO8)
- net SDA: now also U3.6 (GPIO7)
- net TARIFF: now also U3.10 (GPIO10)
- net LED: now reaches R31.1
- net LED: now also U3.5 (GPIO6)
- net at R31.2: now also D1.2 (A); no longer D1.1 (K)
- removed net 5V: DO1.10 (Pin_10), DO1.12 (Pin_12), DO1.2 (Pin_2), DO1.4 (Pin_4), DO1.6 (Pin_6), DO1.8 (Pin_8)
- net ESP/MAINS-1: no longer names the net of X1.2 (Pin_2)
- net ESP/MAINS-1: now also U1.1 (LINE1)
- net ESP/MAINS-2: no longer names the net of X1.1 (Pin_1)
- net ESP/MAINS-2: now also U1.2 (LINE2)
- net VCC renamed +3V3
- net +3V3: now also C2.1, C2.1, C3.1, R5.2, U1.2 (VO), U3.1 (3V3); no longer D1.2 (A)
- new net: C7.2, R5.1, U3.2 (EN/CHIP_PU)
- new net: C21.1, R15.2, U7.3 (+)
- new net: C18.1, R12.2, U5.5 (+)
- new net: R18.1, R24.1, U5.6 (-)
- new net: R22.1, R28.1, U7.6 (-)
- new net: R20.1, R26.1, U6.6 (-)
- new net: R17.1, R23.1, U5.2 (-)
- new net: C17.1, R11.2, U5.3 (+)
- new net: C14.1, R14.1, R8.2
- new net: C16.1, R10.2, R16.1
- new net: C22.1, R16.2, U7.5 (+)
- new net: C11.1, R11.1, R5.2
- new net: R19.1, R25.1, U6.2 (-)
- new net: J12.1 (Pin_1), U3.13 (GPIO18/USB_D-)
- new net: J12.3 (Pin_3), U3.14 (GPIO19/USB_D+)
- new net: C15.1, R15.1, R9.2
- new net: R21.1, R27.1, U7.2 (-)
- new net: C12.1, R12.1, R6.2
- new net: C20.1, R14.2, U6.5 (+)
- new net: C13.1, R13.1, R7.2
- new net: C19.1, R13.2, U6.3 (+)
- new net +12V: C1.1, C10.1, C8.1, C9.1, U1.3 (VI), U1.4 (OUT+), U5.8 (V+), U6.8 (V+), U7.8 (V+)
- new net AOUT0: DO1.2 (Pin_2), R23.2, U5.1
- new net AOUT1: DO1.4 (Pin_4), R24.2, U5.7
- new net AOUT2: DO1.6 (Pin_6), R25.2, U6.1
- new net AOUT3: DO1.8 (Pin_8), R26.2, U6.7
- new net AOUT4: DO1.10 (Pin_10), R27.2, U7.1
- new net AOUT5: DO1.12 (Pin_12), R28.2, U7.7
- new net DOUT0: R5.1, U3.18 (GPIO0/ADC1_CH0/XTAL_32K_P)
- new net DOUT1: R6.1, U3.17 (GPIO1/ADC1_CH1/XTAL_32K_N)
- new net DOUT2: R7.1, U3.16 (GPIO2/ADC1_CH2)
- new net DOUT3: R8.1, U3.15 (GPIO3/ADC1_CH3)
- new net DOUT4: R9.1, U3.3 (GPIO4/ADC1_CH4)
- new net DOUT5: R10.1, U3.4 (GPIO5/ADC2_CH0)
- no-connect marks 4 -> 3
Other:
- removed sheet ESP
- note added: "https://tinyurl.com/2b23mtv8"

Commit message: WIP
Parts:
- C4: footprint Capacitor_SMD:C_1210_3225Metric -> Capacitor_SMD:C_1210_3225Metric_Pad1.33x2.70mm_HandSolder
- R2: footprint Resistor_SMD:R_1206_3216Metric -> Resistor_SMD:R_1206_3216Metric_Pad1.30x1.75mm_HandSolder
Changed lines of the file:
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@@
       (effects (font (size 1.27 1.27)) (justify left))
     )
-    (property "Footprint" "Capacitor_SMD:C_1210_3225Metric" (at 35.56 133.0452 0)
+    (property "Footprint" "Capacitor_SMD:C_1210_3225Metric_Pad1.33x2.70mm_HandSolder" (at 35.56 133.0452 0)
       (effects (font (size 1.27 1.27)) hide)
     )
@@
       (effects (font (size 1.27 1.27)))
     )
-    (property "Footprint" "Resistor_SMD:R_1206_3216Metric" (at 46.99 130.302 90)
+    (property "Footprint" "Resistor_SMD:R_1206_3216Metric_Pad1.30x1.75mm_HandSolder" (at 46.99 130.302 90)
       (effects (font (size 1.27 1.27)) hide)
     )

Commit message: WIP
Other:
- note added: "Next ver: I2C pullup 1k5 replaceMicromatch by IDC replace LM1117 by SMPS"
Changed lines of the file:
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@@
     (effects (font (size 1.524 1.524)) (justify left bottom))
+  )
+  (text "Next ver:\nI2C pullup 1k5\nreplaceMicromatch by IDC\nreplace LM1117 by SMPS" (exclude_from_sim no)
+    (at 110.49 29.21 0)
+    (effects (font (size 1.27 1.27)) (justify left bottom))
   )
   (label "AOUT2" (at 209.55 72.39 0) (fields_autoplaced)

Commit message: WIP
Parts:
- removed C1, C2: 10u, Capacitor_SMD:C_0805_2012Metric, symbol Device:C
- removed C2, C3: 47u, Capacitor_SMD:C_0805_2012Metric, symbol Device:C
- removed U1: LM1117MP-3.3, Package_TO_SOT_SMD:SOT-223-3_TabPin2, symbol Regulator_Linear:LM1117MP-3.3
- added C10: 100u/12V, Capacitor_SMD:CP_Elec_6.3x5.4, symbol Device:C_Polarized
- added C2: 100u/16V, Capacitor_SMD:CP_Elec_6.3x5.4, symbol Device:C_Polarized
- added C4, C7: 100n, Capacitor_SMD:C_0805_2012Metric_Pad1.18x1.45mm_HandSolder, symbol Device:C
- added L2: 6.8uH, Drake:CKCS6028, symbol Device:L
- added R3: 100k, Resistor_SMD:R_0805_2012Metric_Pad1.20x1.40mm_HandSolder, symbol Device:R
- added R6: 30k 1%, Resistor_SMD:R_0805_2012Metric_Pad1.20x1.40mm_HandSolder, symbol Device:R
- added R7: 6.65k 1%, Resistor_SMD:R_0805_2012Metric_Pad1.20x1.40mm_HandSolder, symbol Device:R
- added U3: FR8205, Package_TO_SOT_SMD:SOT-23-6, symbol Drake:FR8205
- DO1: footprint Drake:Micro-Match-FOB-12 -> Connector_IDC:IDC-Header_2x06_P2.54mm_Vertical
- I2C1: footprint Drake:Micro-Match-FOB-4 -> Connector_IDC:IDC-Header_2x03_P2.54mm_Vertical; symbol Drake:I2C -> Drake:I2C-6P
- R29, R30: value 10k -> 1k5
- U3: footprint Espressif:ESP32-C3-WROOM-02 -> Drake:ESP32-C3-WROOM-02 Handsolder
- X1, X2: footprint Drake:DG301-5.0-02 -> Drake:DG235-3.81-02P
Connections:
- net +12V: now also C2.1, C4.2, R3.2, U3.5 (VIN)
- net +3V3: now also C10.1, L2.2, R6.2
- net GND: now also C10.2, C2.2, C4.1, R7.1, U3.2 (GND)
- net at X1.1 (Pin_1): now also U1.1 (LINE1); no longer U1.2 (LINE2)
- net at X1.2 (Pin_2): now also U1.2 (LINE2); no longer U1.1 (LINE1)
- new net: C7.1, U3.1 (BST)
- new net: C7.2, L2.1, U3.6 (LX)
- new net: R6.1, R7.2, U3.3 (FB)
- new net: R3.1, U3.4 (SHDN)
- no-connect marks 3 -> 5
Other:
- note removed: "Next ver: I2C pullup 1k5 replaceMicromatch by IDC replace LM1117 by SMPS"
- moved on the sheet: C10, C11, C12, C13, C14, C15, C16, C17, C18, C19, C20, C21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
