File: ssreg6/board/ssreg6.kicad_pcb (KiCad board)
At the start: 2 copper layers, 45 x 80 mm, 76 parts, among them J1 PROG, J2 Display, U2 FR8205, U3 ESP32-C3-WROOM-02, U4 LM358, U5 LM358, U6 LM358, U7 LTV-354T, X1 12V, X2 TARIFF

Commit message: WIP
Parts:
- moved DO1 5.00 mm to (117.2, 107.7)
- moved I2C1 5.00 mm to (140.7, 107.7)
Other:
- board size 45 x 80 mm -> 45 x 85 mm
Changed lines of the file:
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@@
     (property "ki_keywords" "esp32-c3 module")
     (attr smd)
-    (fp_text reference "U3" (at 0 -13 360) (layer "F.SilkS") hide
+    (fp_text reference "U3" (at 0 -13) (layer "F.SilkS") hide
       (effects (font (size 1 1) (thickness 0.15)))
     )
-    (fp_text value "ESP32-C3-WROOM-02" (at 0 10.5 360) (layer "F.Fab")
+    (fp_text value "ESP32-C3-WROOM-02" (at 0 10.5) (layer "F.Fab")
       (effects (font (size 1 1) (thickness 0.15)))
     )
@@
     (fp_line (start 10.8 9.5) (end 10.8 -12)
       (stroke (width 0.12) (type solid)) (layer "F.CrtYd"))
-    (fp_text user "Antenna Area" (at 0 -8.65 360) (layer "F.SilkS")
+    (fp_text user "Antenna Area" (at 0 -8.65) (layer "F.SilkS")
       (effects (font (size 1 1) (thickness 0.15)))
     )
-    (fp_text user "Antenna Area" (at 0 -8.65 360) (layer "Eco2.User")
+    (fp_text user "Antenna Area" (at 0 -8.65) (layer "Eco2.User")
       (effects (font (size 1 1) (thickness 0.15)))
     )
-    (fp_text user "REF**" (at 0 0 360) (layer "F.Fab")
+    (fp_text user "REF**" (at 0 0) (layer "F.Fab")
       (effects (font (size 1 1) (thickness 0.15)))
     )
@@
     (property "ki_keywords" "connector")
     (attr through_hole)
-    (fp_text reference "X2" (at 0 11 180) (layer "F.SilkS")
+    (fp_text reference "X2" (at 0 11 -180) (layer "F.SilkS")
       (effects (font (size 1 1) (thickness 0.15)))
     )
-    (fp_text value "TARIFF" (at 0.67 14.252 270) (layer "F.SilkS")
+    (fp_text value "TARIFF" (at 0.67 14.252 -90) (layer "F.SilkS")
       (effects (font (size 1 1) (thickness 0.15)) (justify left))
     )
@@
   )
   (footprint "Connector_IDC:IDC-Header_2x03_P2.54mm_Vertical" (layer "F.Cu")
-    (at 140.71 102.71 90)
+    (at 140.71 107.71 90)
     (descr "Through hole IDC box header, 2x03, 2.54mm pitch, DIN 41651 / IEC 60603-13, double rows, https://docs.google.com/spreadsheets/d/16SsEcesNF15N3Lb4niX7dcUr-NY5_MFPQhobNuNppn4/edit#gid=0")
     (tags "Through hole vertical IDC box header THT 2x03 2.54mm double row")
@@
     (property "Sheetname" "")
     (attr through_hole)
-    (fp_text reference "I2C1" (at 1.27 -6.1 270) (layer "F.SilkS") hide
+    (fp_text reference "I2C1" (at 1.27 -6.1 -90) (layer "F.SilkS") hide
       (effects (font (size 1 1) (thickness 0.15)))
     )
-    (fp_text value "I2C" (at 7.71 2.54 360) (layer "F.SilkS")
+    (fp_text value "I2C" (at 7.71 2.54) (layer "F.SilkS")
       (effects (font (size 1 1) (thickness 0.15)))
     )
@@
     (fp_line (start -3.18 10.18) (end -3.18 -4.1)
       (stroke (width 0.1) (type solid)) (layer "F.Fab"))
-    (fp_text user "${REFERENCE}" (at 1.27 2.54 360) (layer "F.Fab")
+    (fp_text user "${REFERENCE}" (at 1.27 2.54) (layer "F.Fab")
       (effects (font (size 1 1) (thickness 0.15)))
     )
@@
     (property "ki_keywords" "connector")
     (attr through_hole)
-    (fp_text reference "X1" (at 0 11 180) (layer "F.SilkS")
+    (fp_text reference "X1" (at 0 11 -180) (layer "F.SilkS")
       (effects (font (size 1 1) (thickness 0.15)))
     )
-    (fp_text value "12V" (at 2 18.052 270) (layer "F.SilkS")
+    (fp_text value "12V" (at 2 18.052 -90) (layer "F.SilkS")
       (effects (font (size 1 1) (thickness 0.15)) (justify right))
     )
@@
     (property "ki_keywords" "cap capacitor")
     (attr smd)
-    (fp_text reference "C3" (at 3.5 0 360) (layer "F.SilkS")
+    (fp_text reference "C3" (at 3.5 0) (layer "F.SilkS")
       (effects (font (size 1 1) (thickness 0.15)))
     )
-    (fp_text value "100n" (at 0 1.68 360) (layer "F.Fab")
+    (fp_text value "100n" (at 0 1.68) (layer "F.Fab")
       (effects (font (size 1 1) (thickness 0.15)))
     )
@@
     (fp_line (start 1 0.625) (end -1 0.625)
       (stroke (width 0.1) (type solid)) (layer "F.Fab"))
-    (fp_text user "${REFERENCE}" (at 0 0 360) (layer "F.Fab")
+    (fp_text user "${REFERENCE}" (at 0 0) (layer "F.Fab")
       (effects (font (size 0.5 0.5) (thickness 0.08)))
     )
@@
   )
   (footprint "Connector_IDC:IDC-Header_2x06_P2.54mm_Vertical" (layer "F.Cu")
-    (at 117.15 102.71 90)
+    (at 117.15 107.71 90)
     (descr "Through hole IDC box header, 2x06, 2.54mm pitch, DIN 41651 / IEC 60603-13, double rows, https://docs.google.com/spreadsheets/d/16SsEcesNF15N3Lb4niX7dcUr-NY5_MFPQhobNuNppn4/edit#gid=0")
     (tags "Through hole vertical IDC box header THT 2x06 2.54mm double row")
@@
   (gr_line (start 109 26) (end 154 26)
     (stroke (width 0.1) (type default)) (layer "Edge.Cuts"))
-  (gr_line (start 154 106) (end 109 106)
+  (gr_line (start 154 111) (end 109 111)
     (stroke (width 0.1) (type default)) (layer "Edge.Cuts"))
   (gr_line (start 109 106) (end 109 26)
@@
   (gr_line (start 154 26) (end 154 106)
     (stroke (width 0.1) (type default)) (layer "Edge.Cuts"))
-  (gr_text "A4" (at 127.33 95.5) (layer "F.SilkS")
+  (gr_text "A4" (at 127.33 101) (layer "F.SilkS")
     (effects (font (size 1 1) (thickness 0.25) bold) (justify bottom))
   )
-  (gr_text "A2" (at 122.25 95.5) (layer "F.SilkS")
+  (gr_text "A2" (at 122.25 101) (layer "F.SilkS")
     (effects (font (size 1 1) (thickness 0.25) bold) (justify bottom))
   )
-  (gr_text "A3" (at 124.79 95.5) (layer "F.SilkS")
+  (gr_text "A3" (at 124.79 101) (layer "F.SilkS")
     (effects (font (size 1 1) (thickness 0.25) bold) (justify bottom))
   )
-  (gr_text "A1" (at 119.71 95.5) (layer "F.SilkS")
+  (gr_text "A1" (at 119.71 101) (layer "F.SilkS")
     (effects (font (size 1 1) (thickness 0.25) bold) (justify bottom))
   )
-  (gr_text "A5" (at 129.87 95.5) (layer "F.SilkS")
+  (gr_text "A5" (at 129.87 101) (layer "F.SilkS")
     (effects (font (size 1 1) (thickness 0.25) bold) (justify bottom))
   )
-  (gr_text "A0" (at 117.17 95.5) (layer "F.SilkS")
+  (gr_text "A0" (at 117.17 101) (layer "F.SilkS")
     (effects (font (size 1 1) (thickness 0.25) bold) (justify bottom))
   )
@@
   )
   (dimension (type aligned) (layer "Dwgs.User")
-    (pts (xy 109 106) (xy 109 26))
+    (pts (xy 109 111) (xy 109 26))
     (height -17)
-    (gr_text "80,0000 mm" (at 90.85 66 90) (layer "Dwgs.User")
+    (gr_text "85,0000 mm" (at 90.85 68.5 90) (layer "Dwgs.User")
       (effects (font (size 1 1) (thickness 0.15)))
     )
@@
         (xy 109 26.021216)
         (xy 154 25.996464)
-        (xy 154 106)
-        (xy 109 106)
+        (xy 154 111)
+        (xy 109 111)
       )
     )

Commit message: library update
Parts:
- U3: footprint Drake:ESP32-C3-WROOM-02 Handsolder -> Drake:ESP32-C3-WROOM-02-Handsolder

Commit message: board WIP
Parts:
- J2: value Display -> AUX; footprint Connector_PinHeader_2.54mm:PinHeader_1x03_P2.54mm_Vertical -> Connector_PinHeader_2.54mm:PinHeader_1x05_P2.54mm_Vertical
- moved C21 91.5 mm to (146.0, 44.0), turned to 0 degrees
- moved R35 86.8 mm to (146.0, 49.0), turned to 180 degrees
- moved U7 75.9 mm to (152.0, 47.0), turned to -90 degrees
- moved R1 75.0 mm to (112.0, 57.0), turned to -90 degrees
- moved R37 73.1 mm to (137.0, 108.0), turned to -90 degrees
- moved R2 71.8 mm to (133.5, 55.0), turned to 180 degrees
- moved R36 71.7 mm to (137.0, 104.0), turned to -90 degrees
- moved C1 71.5 mm to (112.0, 53.0)
- moved C2 70.5 mm to (127.5, 58.0), turned to -90 degrees
- moved C22 69.5 mm to (147.0, 54.0)
- moved R3 68.9 mm to (141.0, 52.0), turned to 0 degrees
- moved R4 68.8 mm to (138.0, 55.0), turned to 0 degrees
- moved R40 68.6 mm to (147.0, 57.0)
- moved R39 68.5 mm to (152.0, 54.0)
- moved C3 65.8 mm to (133.0, 59.0), turned to 90 degrees
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Connections:
- J2 pad 2: /DISP -> /AUX0
- J2 pad 3: +3V3 -> /AUX1
- U3 pad 11: unconnected-(U3-GPIO20/U0RXD-Pad11) -> /AUX0
- U3 pad 12: /DISP -> /AUX1
- U3 pad 8: unconnected-(U3-GPIO9-Pad8) -> /AUX2
Routing:
- net +3V3: track 0.00 -> 156.9 mm, vias 0 -> 4
- net /SDA: track 0.00 -> 104.9 mm
- net /AUX2: track 0.00 -> 93.7 mm, vias 0 -> 2
- net /SCL: track 0.00 -> 91.5 mm
- net /DOUT5: track 0.00 -> 82.7 mm, vias 0 -> 2
- net /AUX0: track 0.00 -> 81.0 mm, vias 0 -> 1
- net +12V: track 0.00 -> 79.4 mm, vias 0 -> 2
- net /AUX1: track 0.00 -> 78.6 mm, vias 0 -> 1
- net /DOUT3: track 0.00 -> 69.1 mm, vias 0 -> 2
- net /DOUT4: track 0.00 -> 64.7 mm
- net /DOUT1: track 0.00 -> 61.5 mm, vias 0 -> 2
- net /TARIFF: track 0.00 -> 57.0 mm, vias 0 -> 1
- net /AOUT1: track 0.00 -> 57.0 mm, vias 0 -> 2
- net /DOUT2: track 0.00 -> 52.5 mm, vias 0 -> 4
- net /AOUT0: track 0.00 -> 48.5 mm, vias 0 -> 1
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Other:
- board size 45 x 85 mm -> 48 x 86 mm
- board text added: "+"
- board text added: "-"
- board text added: "AccuWatt SSREG6 v2.2"
- board text removed: "AccuWatt SSREG6 v2.2 drake.cz"
