File: fanctrl/board/fanctrl.kicad_pcb (KiCad board)
At the start: 2 copper layers, 45 x 85 mm, 25 parts, among them J1 PROG, J2 Display, J5 Fan1, Q1 BXT420N03M, U2 FR8205, U3 ESP32-C3-WROOM-02, X1 12V

Commit message: fanctrl schema
Parts:
- added D3: SK22, Diode_SMD:D_SMB_Handsoldering, F.Cu at (50.9, 53.3)
- added D4: SK22, Diode_SMD:D_SMB_Handsoldering, F.Cu at (34.3, 53.3)
- added J3: Fan1, Drake:DG235-3.81-02P, F.Cu at (32.9, 38.4)
- added Q2: YJM04N10A, Package_TO_SOT_SMD:SOT-223, F.Cu at (44.1, 38.7)
- added Q3: YJM04N10A, Package_TO_SOT_SMD:SOT-223, F.Cu at (34.0, 60.3)
- added R10: 100, Resistor_SMD:R_0805_2012Metric_Pad1.20x1.40mm_HandSolder, F.Cu at (41.2, 60.5)
- added R7: 10k, Resistor_SMD:R_0805_2012Metric_Pad1.20x1.40mm_HandSolder, F.Cu at (48.0, 57.5)
- added R8: 100, Resistor_SMD:R_0805_2012Metric_Pad1.20x1.40mm_HandSolder, F.Cu at (48.0, 60.5)
- added R9: 10k, Resistor_SMD:R_0805_2012Metric_Pad1.20x1.40mm_HandSolder, F.Cu at (41.2, 57.5)
- Q1: value BXT420N03M -> YJM04N10A; footprint Package_TO_SOT_SMD:SOT-23 -> Package_TO_SOT_SMD:SOT-223
Connections:
- J5 pad 1: Net-(D2-A) -> /Driver/SW_GND
- Q1 pad 2: GND -> /Driver/SW_GND
- Q1 pad 3: Net-(D2-A) -> GND
- R5 pad 2: /FAN_1 -> Net-(R5-Pad2)
- R6 pad 1: /FAN_1 -> Net-(R5-Pad2)
- R6 pad 2: Net-(Q1-G) -> Net-(Q2-G)

Commit message: board design
Parts:
- removed D2: SK22, Diode_SMD:D_SMB_Handsoldering
- removed Q2: YJM04N10A, Package_TO_SOT_SMD:SOT-223
- removed R5: 10k, Resistor_SMD:R_0805_2012Metric_Pad1.20x1.40mm_HandSolder
- removed R6: 100, Resistor_SMD:R_0805_2012Metric_Pad1.20x1.40mm_HandSolder
- J2: value Display -> AUX; footprint Connector_PinHeader_2.54mm:PinHeader_1x03_P2.54mm_Vertical -> Connector_PinHeader_2.54mm:PinHeader_1x05_P2.54mm_Vertical
- J3: value Fan1 -> Fan2
- moved J3 108.5 mm to (121.9, 100.3)
- moved D4 99.4 mm to (125.0, 94.0), turned to 180 degrees
- moved Q3 93.7 mm to (124.0, 86.0), turned to -90 degrees
- moved R10 86.5 mm to (126.0, 78.0), turned to -90 degrees
- moved R9 83.3 mm to (122.0, 78.0), turned to 90 degrees
- moved D3 75.9 mm to (115.0, 94.0), turned to 180 degrees
- moved R1 72.6 mm to (114.5, 57.0), turned to -90 degrees
- moved R8 71.2 mm to (117.0, 78.0), turned to -90 degrees
- moved J5 69.4 mm to (114.3, 100.3)
- moved C1 69.1 mm to (114.5, 53.0)
- moved R7 68.1 mm to (113.0, 78.0), turned to 90 degrees
- moved R36 66.5 mm to (136.0, 97.0), turned to 0 degrees
- moved R2 66.0 mm to (139.5, 55.0), turned to 180 degrees
- moved R3 64.0 mm to (144.0, 57.5), turned to 0 degrees
- moved R4 63.1 mm to (144.0, 55.0), turned to 0 degrees
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Connections:
- J2 pad 2: /DISP -> /AUX0
- J2 pad 3: +3V3 -> /AUX1
- U3 pad 11: unconnected-(U3-GPIO20/U0RXD-Pad11) -> /AUX0
- U3 pad 12: /DISP -> /AUX1
- U3 pad 16: unconnected-(U3-GPIO2/ADC1_CH2-Pad16) -> /AUX2
Routing:
- net +3V3: track 0.00 -> 151.1 mm
- net +12V: track 0.00 -> 101.7 mm
- net /SDA: track 0.00 -> 96.5 mm, vias 0 -> 4
- net /SCL: track 0.00 -> 72.4 mm, vias 0 -> 4
- net /FAN_1: track 0.00 -> 58.8 mm
- net /FAN_2: track 0.00 -> 55.8 mm
- net GND: track 0.00 -> 39.3 mm, vias 0 -> 69
- net /AUX0: track 0.00 -> 34.1 mm, vias 0 -> 2
- net /AUX2: track 0.00 -> 33.4 mm, vias 0 -> 2
- net /AUX1: track 0.00 -> 32.8 mm, vias 0 -> 2
- net Net-(U3-EN/CHIP_PU): track 0.00 -> 24.9 mm, vias 0 -> 2
- net /Driver/SW_GND: track 0.00 -> 24.4 mm
- net /LED: track 0.00 -> 24.4 mm, vias 0 -> 2
- net /Driver1/SW_GND: track 0.00 -> 23.4 mm
- net Net-(J1-Pin_3): track 0.00 -> 12.2 mm
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Other:
- board size 45 x 85 mm -> 40 x 86 mm
- board text added: "+"
- board text added: "AccuWatt FANCTRL v1.0 drake.cz"
- board text removed: "A0"
- board text removed: "A1"
- board text removed: "A2"
- board text removed: "A3"
- board text removed: "A4"
- board text removed: "A5"
- board text removed: "AccuWatt SSREG6 v2.2 drake.cz"

Commit message: ceramic capacitors on PSU & JLC order
Parts:
- removed U2: FR8205, Package_TO_SOT_SMD:SOT-23-6
- added C6: 10u/16V, Capacitor_SMD:C_0805_2012Metric_Pad1.18x1.45mm_HandSolder, F.Cu at (142.0, 74.0)
- added C7: 10u/16V, Capacitor_SMD:C_0805_2012Metric_Pad1.18x1.45mm_HandSolder, F.Cu at (142.0, 76.0)
- added C8: 100u/16V, Capacitor_SMD:CP_Elec_6.3x5.4, F.Cu at (142.0, 75.0)
- added U1: FR8205, Package_TO_SOT_SMD:SOT-23-6, F.Cu at (139.5, 58.5)
- C3, C4: value 100n -> 10u/16V
- C5: value 100u/12V -> 100n; footprint Capacitor_SMD:CP_Elec_6.3x5.4 -> Capacitor_SMD:C_0805_2012Metric_Pad1.18x1.45mm_HandSolder
- moved C5 13.2 mm to (139.5, 62.0)
- moved C4 12.5 mm to (140.5, 49.5), turned to 0 degrees
- moved C3 5.10 mm to (140.5, 47.5), turned to 0 degrees
- moved C2 1.50 mm to (140.5, 48.5)
Connections:
- C3 pad 1: GND -> +12V
- C3 pad 2: +12V -> GND
- C4 pad 1: Net-(U2-BST) -> +12V
- C4 pad 2: Net-(U2-LX) -> GND
- C5 pad 1: +3V3 -> Net-(U1-BST)
- C5 pad 2: GND -> Net-(U1-LX)
- L1 pad 1: Net-(U2-LX) -> Net-(U1-LX)
Routing:
- net Net-(U2-LX): track 7.36 -> 0.00 mm
- net Net-(U1-LX): track 0.00 -> 7.36 mm
- net GND: track 39.3 -> 36.6 mm
- net Net-(U2-BST): track 2.59 -> 0.00 mm
- net Net-(U1-BST): track 0.00 -> 2.59 mm
